Commit message: add Catersian goal pose control

File: dvrk_env/dvrk_description/psm/psm_for_issacgym.urdf (robot description, URDF)
Before this commit: robot psm, 12 links, 11 joints
Joints:
- joint psm_rev_joint: limit lower=-1.57 upper=1.57 effort=1000 velocity=10 -> lower=0 upper=0 effort=1000 velocity=10

Commit message: add collision object to MoveIt scene, add preshape generator, add straight-line server

File: dvrk_env/dvrk_description/psm/psm_for_issacgym.urdf (robot description, URDF)
Before this commit: robot psm, 12 links, 11 joints
Joints:
- joint psm_main_insertion_joint: limit lower=0.0 upper=0.24 effort=1000.0 velocity=0.001 -> lower=0.0 upper=0.24 effort=1000.0 velocity=0.0000000000001

Commit message: fix point cloud generation of a soft object. Also see point_cloud_test_soft.py

File: dvrk_env/dvrk_description/psm/psm_for_issacgym.urdf (robot description, URDF)
Before this commit: robot psm, 12 links, 11 joints
Joints:
- joint psm_tool_roll_joint: limit lower=-3.14159 upper=3.14159 effort=1000.0 velocity=10.0 -> lower=-3.14 upper=3.14 effort=1000.0 velocity=10.0

Commit message: commit before transfering to tars machine

File: dvrk_env/dvrk_description/psm/psm_for_issacgym.urdf (robot description, URDF)
Before this commit: robot psm, 12 links, 11 joints
Joints:
- joint psm_tool_gripper1_joint: limit lower=-1.0 upper=1.0 effort=1 velocity=0.1 -> lower=-1.0 upper=2.0 effort=1 velocity=0.1
- joint psm_tool_gripper2_joint: limit lower=-1.0 upper=1.0 effort=1 velocity=0.1 -> lower=-1.0 upper=2.0 effort=1 velocity=0.1
